Commit message: '111'

File: src/hexapod/robot/hexapod.urdf (robot description, URDF)
Before this commit: robot Hexapod, 32 links, 31 joints
Links:
- added link world
Joints:
- added joint world_connect: type fixed, parent world, child base_link, origin xyz=0 0 0.1 rpy=0 0 0

File: src/hexapod/robot/hexapod.xacro (robot description, xacro)
@@ -3,4 +3,10 @@
   <xacro:include filename="/home/jichen/paper11_ws/src/hexapod/robot/hexapod_urdf.xacro" />
   <!-- <xacro:arg name="arm_id_1" default="panda_1" /> -->
+  <link name="world"/>
+  <joint name="world_connect" type="fixed">
+    <parent link="world"/>
+    <child link="base_link"/>
+    <origin xyz="0 0 0.1" rpy="0 0 0" />
+  </joint>
   <link name="base_link"/>
     <xacro:hexapod parent="base_link">

Commit message: data

File: src/hexapod/robot/hexapod.urdf (robot description, URDF)
Before this commit: robot Hexapod, 33 links, 32 joints
Joints:
- joint j_c1_lf: limit lower=-2.6179939 upper=2.6179939 effort=5.8 velocity=5.6548668 -> lower=-2.6179939 upper=2.6179939 effort=5.8 velocity=10
- joint j_c1_lm: limit lower=-2.6179939 upper=2.6179939 effort=5.8 velocity=5.6548668 -> lower=-2.6179939 upper=2.6179939 effort=5.8 velocity=10
- joint j_c1_lr: limit lower=-2.6179939 upper=2.6179939 effort=5.8 velocity=5.6548668 -> lower=-2.6179939 upper=2.6179939 effort=5.8 velocity=10
- joint j_c1_rf: limit lower=-2.6179939 upper=2.6179939 effort=5.8 velocity=5.6548668 -> lower=-2.6179939 upper=2.6179939 effort=5.8 velocity=10
- joint j_c1_rm: limit lower=-2.6179939 upper=2.6179939 effort=5.8 velocity=5.6548668 -> lower=-2.6179939 upper=2.6179939 effort=5.8 velocity=10
- joint j_c1_rr: limit lower=-2.6179939 upper=2.6179939 effort=5.8 velocity=5.6548668 -> lower=-2.6179939 upper=2.6179939 effort=5.8 velocity=10
- joint j_thigh_lf: limit lower=-2.6179939 upper=2.6179939 effort=5.8 velocity=5.6548668 -> lower=-2.6179939 upper=2.6179939 effort=5.8 velocity=10
- joint j_thigh_lm: limit lower=-2.6179939 upper=2.6179939 effort=5.8 velocity=5.6548668 -> lower=-2.6179939 upper=2.6179939 effort=5.8 velocity=10
- joint j_thigh_lr: limit lower=-2.6179939 upper=2.6179939 effort=5.8 velocity=5.6548668 -> lower=-2.6179939 upper=2.6179939 effort=5.8 velocity=10
- joint j_thigh_rf: limit lower=-2.6179939 upper=2.6179939 effort=5.8 velocity=5.6548668 -> lower=-2.6179939 upper=2.6179939 effort=5.8 velocity=10
- joint j_thigh_rm: limit lower=-2.6179939 upper=2.6179939 effort=5.8 velocity=5.6548668 -> lower=-2.6179939 upper=2.6179939 effort=5.8 velocity=10
- joint j_thigh_rr: limit lower=-2.6179939 upper=2.6179939 effort=5.8 velocity=5.6548668 -> lower=-2.6179939 upper=2.6179939 effort=5.8 velocity=10
- joint j_tibia_lf: limit lower=-1.0 upper=1.0 effort=5.8 velocity=5.6548668 -> lower=-2.5 upper=2.5 effort=5.8 velocity=10
- joint j_tibia_lm: limit lower=-1.0 upper=1.0 effort=5.8 velocity=5.6548668 -> lower=-2.5 upper=2.5 effort=5.8 velocity=10
- joint j_tibia_lr: limit lower=-1.0 upper=1.0 effort=5.8 velocity=5.6548668 -> lower=-2.5 upper=2.5 effort=5.8 velocity=10
- joint j_tibia_rf: limit lower=-1.0 upper=1.0 effort=5.8 velocity=5.6548668 -> lower=-2.5 upper=2.5 effort=5.8 velocity=10
- joint j_tibia_rm: limit lower=-1.0 upper=1.0 effort=5.8 velocity=5.6548668 -> lower=-2.5 upper=2.5 effort=5.8 velocity=10
- joint j_tibia_rr: limit lower=-1.0 upper=1.0 effort=5.8 velocity=5.6548668 -> lower=-2.5 upper=2.5 effort=5.8 velocity=10

File: src/hexapod/robot/hexapod_urdf.xacro (robot description, xacro)
@@ -209,5 +209,5 @@
     <origin xyz="0 0 0" rpy="${r1p1y1}" />
     <axis xyz="0 0 -1" />
-    <limit effort="5.8" velocity="5.6548668" lower="-2.6179939" upper="2.6179939" />
+    <limit effort="5.8" velocity="10" lower="-2.6179939" upper="2.6179939" />
     <dynamics damping="0.5" friction="0.0" />
   </joint>
@@ -217,5 +217,5 @@
     <origin xyz="0 0.053 0" rpy="${M_PI/2} 0 ${M_PI/2}" />
     <axis xyz="0 0 1" />
-    <limit effort="5.8" velocity="5.6548668" lower="-2.6179939" upper="2.6179939" />
+    <limit effort="5.8" velocity="10" lower="-2.6179939" upper="2.6179939" />
     <dynamics damping="0.5" friction="0.0" />
   </joint>
@@ -226,5 +226,5 @@
     <origin rpy="3.141592653589793 0 3.141592653589793" xyz="0.0525 0 0"/>
     <axis xyz="0 0 -1" />
-    <limit effort="5.8" velocity="5.6548668" lower="-1.0" upper="1.0" />
+    <limit effort="5.8" velocity="10" lower="-2.5" upper="2.5" />
     <dynamics damping="0.5" friction="0.0" />
   </joint>

Commit message: data

File: src/hexapod/robot/hexapod.urdf (robot description, URDF)
Before this commit: robot Hexapod, 33 links, 32 joints
Joints:
- joint j_c1_lf: origin xyz=0 0 0 rpy=0 3.141592653589793 3.141592653589793 -> xyz=0 0 0 rpy=0 3.141592653589793 4.1887902047863905
- joint j_c1_lr: origin xyz=0 0 0 rpy=0 3.141592653589793 3.141592653589793 -> xyz=0 0 0 rpy=0 3.141592653589793 2.0943951023931957
- joint j_c1_rf: origin xyz=0 0 0 rpy=0 3.141592653589793 0 -> xyz=0 0 0 rpy=0 3.141592653589793 -1.0471975511965976
- joint j_c1_rr: origin xyz=0 0 0 rpy=0 3.141592653589793 0 -> xyz=0 0 0 rpy=0 3.141592653589793 1.0471975511965976
- joint j_thigh_lf: origin xyz=0 0.053 0 rpy=1.5707963267948966 0 1.5707963267948966 -> xyz=0 0.053 0 rpy=1.5707963267948966 -0.2617993877991494 1.5707963267948966
- joint j_thigh_lm: origin xyz=0 0.053 0 rpy=1.5707963267948966 0 1.5707963267948966 -> xyz=0 0.053 0 rpy=1.5707963267948966 -0.2617993877991494 1.5707963267948966
- joint j_thigh_lr: origin xyz=0 0.053 0 rpy=1.5707963267948966 0 1.5707963267948966 -> xyz=0 0.053 0 rpy=1.5707963267948966 -0.2617993877991494 1.5707963267948966
- joint j_thigh_rf: origin xyz=0 0.053 0 rpy=1.5707963267948966 0 1.5707963267948966 -> xyz=0 0.053 0 rpy=1.5707963267948966 -0.2617993877991494 1.5707963267948966
- joint j_thigh_rm: origin xyz=0 0.053 0 rpy=1.5707963267948966 0 1.5707963267948966 -> xyz=0 0.053 0 rpy=1.5707963267948966 -0.2617993877991494 1.5707963267948966
- joint j_thigh_rr: origin xyz=0 0.053 0 rpy=1.5707963267948966 0 1.5707963267948966 -> xyz=0 0.053 0 rpy=1.5707963267948966 -0.2617993877991494 1.5707963267948966
- joint j_tibia_lf: origin xyz=0.0525 0 0 rpy=3.141592653589793 0 3.141592653589793 -> xyz=0.0525 0 0 rpy=3.141592653589793 0 2.0943951023931953
- joint j_tibia_lm: origin xyz=0.0525 0 0 rpy=3.141592653589793 0 3.141592653589793 -> xyz=0.0525 0 0 rpy=3.141592653589793 0 2.0943951023931953
- joint j_tibia_lr: origin xyz=0.0525 0 0 rpy=3.141592653589793 0 3.141592653589793 -> xyz=0.0525 0 0 rpy=3.141592653589793 0 2.0943951023931953
- joint j_tibia_rf: origin xyz=0.0525 0 0 rpy=3.141592653589793 0 3.141592653589793 -> xyz=0.0525 0 0 rpy=3.141592653589793 0 2.0943951023931953
- joint j_tibia_rm: origin xyz=0.0525 0 0 rpy=3.141592653589793 0 3.141592653589793 -> xyz=0.0525 0 0 rpy=3.141592653589793 0 2.0943951023931953
- joint j_tibia_rr: origin xyz=0.0525 0 0 rpy=3.141592653589793 0 3.141592653589793 -> xyz=0.0525 0 0 rpy=3.141592653589793 0 2.0943951023931953

File: src/hexapod/robot/hexapod_urdf.xacro (robot description, xacro)
@@ -44,10 +44,10 @@
         <material>Gazebo/Grey</material>
       </gazebo>
-    <xacro:leg_l xyz="0.038 0.046 0.02"  rpy="0 ${M_PI} ${-M_PI/2}" r1p1y1="0 ${M_PI} 0" suffix="rf"/>
+    <xacro:leg_l xyz="0.038 0.046 0.02"  rpy="0 ${M_PI} ${-M_PI/2}" r1p1y1="0 ${M_PI} ${-M_PI/3}" suffix="rf"/>
     <xacro:leg_l xyz="0.038 0.0  0.02"  rpy="0 ${M_PI} ${-M_PI/2}" r1p1y1="0 ${M_PI} 0" suffix="rm"/>
-    <xacro:leg_l xyz="0.038 -0.046  0.02"  rpy="0 ${M_PI} ${-M_PI/2}" r1p1y1="0 ${M_PI} 0" suffix="rr"/>
-    <xacro:leg_l xyz="-0.038 0.046  0.02"  rpy="0 ${-M_PI} ${3*M_PI/2}" r1p1y1="0 ${M_PI} ${M_PI}" suffix="lf"/>
+    <xacro:leg_l xyz="0.038 -0.046  0.02"  rpy="0 ${M_PI} ${-M_PI/2}" r1p1y1="0 ${M_PI} ${M_PI/3}" suffix="rr"/>
+    <xacro:leg_l xyz="-0.038 0.046  0.02"  rpy="0 ${-M_PI} ${3*M_PI/2}" r1p1y1="0 ${M_PI} ${M_PI + M_PI/3}" suffix="lf"/>
     <xacro:leg_l xyz="-0.038 0.0  0.02"  rpy="0 ${-M_PI} ${3*M_PI/2}" r1p1y1="0 ${M_PI} ${M_PI}" suffix="lm"/>
-    <xacro:leg_l xyz="-0.038 -0.046  0.02"  rpy="0 ${-M_PI} ${3*M_PI/2}" r1p1y1="0 ${M_PI} ${M_PI}" suffix="lr"/>
+    <xacro:leg_l xyz="-0.038 -0.046  0.02"  rpy="0 ${-M_PI} ${3*M_PI/2}" r1p1y1="0 ${M_PI} ${M_PI - M_PI/3}" suffix="lr"/>
 </xacro:macro>
  <xacro:macro name="utilities" params="xyz rpy">
@@ -215,5 +215,5 @@
     <parent link="c1_${suffix}"/>
     <child link="thigh_${suffix}"/>
-    <origin xyz="0 0.053 0" rpy="${M_PI/2} 0 ${M_PI/2}" />
+    <origin xyz="0 0.053 0" rpy="${M_PI/2} ${-M_PI/12} ${M_PI/2}" />
     <axis xyz="0 0 1" />
     <limit effort="5.8" velocity="10" lower="-2.6179939" upper="2.6179939" />
@@ -224,5 +224,5 @@
     <child link="tibia_${suffix}"/>
     <!-- <origin xyz="0 ${thigh_offset_y} ${thigh_offset_z}" rpy="-1.5707 0 3.14159" /> -->
-    <origin rpy="3.141592653589793 0 3.141592653589793" xyz="0.0525 0 0"/>
+    <origin rpy="3.141592653589793 0 ${2*M_PI/3}" xyz="0.0525 0 0"/>
     <axis xyz="0 0 -1" />
     <limit effort="5.8" velocity="10" lower="-2.5" upper="2.5" />

Commit message: data

File: src/hexapod/robot/hexapod.urdf (robot description, URDF)
Before this commit: robot Hexapod, 33 links, 32 joints
Links:
- removed link world
Joints:
- removed joint world_connect

File: src/hexapod/robot/hexapod.xacro (robot description, xacro)
@@ -3,10 +3,10 @@
   <xacro:include filename="/home/jichen/paper11_ws/src/hexapod/robot/hexapod_urdf.xacro" />
   <!-- <xacro:arg name="arm_id_1" default="panda_1" /> -->
-  <link name="world"/>
+  <!-- <link name="world"/>
   <joint name="world_connect" type="fixed">
     <parent link="world"/>
     <child link="base_link"/>
     <origin xyz="0 0 0.1" rpy="0 0 0" />
-  </joint>
+  </joint> -->
   <link name="base_link"/>
     <xacro:hexapod parent="base_link">

Commit message: data

File: src/hexapod/robot/hexapod.urdf (robot description, URDF)
Before this commit: robot Hexapod, 32 links, 31 joints
Links:
- added link world
Joints:
- added joint world_connect: type fixed, parent world, child base_link, origin xyz=0 0 0.1 rpy=0 0 0

File: src/hexapod/robot/hexapod.xacro (robot description, xacro)
@@ -3,10 +3,10 @@
   <xacro:include filename="/home/jichen/paper11_ws/src/hexapod/robot/hexapod_urdf.xacro" />
   <!-- <xacro:arg name="arm_id_1" default="panda_1" /> -->
-  <!-- <link name="world"/>
+  <link name="world"/>
   <joint name="world_connect" type="fixed">
     <parent link="world"/>
     <child link="base_link"/>
     <origin xyz="0 0 0.1" rpy="0 0 0" />
-  </joint> -->
+  </joint>
   <link name="base_link"/>
     <xacro:hexapod parent="base_link">
